Commit message: Rename bugv_rtab node to not have the map. Update bugv urdf to correct build and tested! #14

File: ros/src/bugv_rtab/urdf/bugv.urdf (robot description, URDF)
Before this commit: robot bugv, 4 links, 3 joints
Links:
- removed link zed_description
- added link zed_camera_center
Joints:
- joint px4_joint: origin xyz=-0.08 0 0 rpy=0 0 -1.5707963267 -> xyz=-0.08 0 0 rpy=0 0 1.5707963267
- joint zed_joint: child zed_description -> zed_camera_center
