Commit message: Update URDF to align rplidar frame with robot. mapping is working.

File: ros/src/bugv/urdf/bugv.urdf (robot description, URDF)
Before this commit: robot bugv, 4 links, 3 joints
Joints:
- joint lidar_joint: origin xyz=0.105 -0.105 0.03 rpy=0 0 0 -> xyz=0.105 -0.105 0.03 rpy=0 0 3.1415926536

Commit message: Remove bugv_tf node as it is replaced by the URDF.

File: ros/src/bugv/urdf/bugv.urdf (robot description, URDF)
Before this commit: robot bugv, 4 links, 3 joints
Links:
- added link zed_imu_link
- added link zed_left_camera_frame
- added link zed_left_camera_optical_frame
- added link zed_right_camera_frame
- added link zed_right_camera_optical_frame
- link zed_camera_center: geometry visual mesh filename=package://zed_wrapper/urdf/models/ZEDM.stl
Joints:
- added joint imu_link_joint: type floating, parent zed_camera_center, child zed_imu_link, origin xyz=0 0 0 rpy=0 0 0
- added joint zed_left_camera_joint: type fixed, parent zed_camera_center, child zed_left_camera_frame, origin xyz=0 0.03 0 rpy=0 0 0
- added joint zed_left_camera_optical_joint: type fixed, parent zed_left_camera_frame, child zed_left_camera_optical_frame, origin xyz=0 0 0 rpy=-1.57079632679 0.0 -1.57079632679
- added joint zed_right_camera_joint: type fixed, parent zed_camera_center, child zed_right_camera_frame, origin xyz=0 -0.03 0 rpy=0 0 0
- added joint zed_right_camera_optical_joint: type fixed, parent zed_right_camera_frame, child zed_right_camera_optical_frame, origin xyz=0 0 0 rpy=-1.57079632679 0.0 -1.57079632679

Commit message: Update urdf to correctly display the height of the frames of the robot

File: ros/src/bugv/urdf/bugv.urdf (robot description, URDF)
Before this commit: robot bugv, 9 links, 8 joints
Links:
- added link base_plate
Joints:
- added joint base_joint: type fixed, parent base_link, child base_plate, origin xyz=0 0 0.15 rpy=0 0 0
- joint lidar_joint: parent base_link -> base_plate
- joint px4_joint: parent base_link -> base_plate
- joint zed_joint: parent base_link -> base_plate
